Commit message: fixed ros2 controllers and tested the connection between mujoco and ROS

File: workspace/src/dobot_description/urdf/cr5/cr5.urdf.xacro (robot description, xacro)
@@ -2,7 +2,7 @@
 <robot xmlns:xacro="http://www.ros.org/wiki/xacro" name="cr5">
     <xacro:arg name="prefix" default="" />
-    <xacro:arg name="package_name" default="cr5_description" />
-    <xacro:include filename="$(find ${package_name})/urdf/macro.xacro" />
-    <xacro:include filename="$(find ${package_name})/urdf/controller.xacro" />
+    <xacro:arg name="mujoco_model" default="$(find dobot_mujoco_integration)/scenes/main_scene.xml" />
+    <xacro:include filename="$(find dobot_description)/urdf/cr5/cr5_macro.xacro" />
+    <xacro:include filename="$(find dobot_description)/urdf/cr5/cr5_controller.xacro" />
     <link name="world" />
     <joint name="$(arg prefix)world_to_base_joint" type="fixed">
@@ -11,5 +11,5 @@
         <origin xyz="0 0 0" rpy="0 0 0" />
     </joint>
-    <xacro:cr5_robot prefix="$(arg prefix)" package_name="$(arg package_name)" />
-    <xacro:cr5_ros2_control name="CR5HardwareInterface" prefix="$(arg prefix)" />
+    <xacro:cr5_robot prefix="$(arg prefix)" />
+    <xacro:cr5_ros2_control prefix="$(arg prefix)" mujoco_model="$(arg mujoco_model)" />
 </robot>

File: workspace/src/dobot_description/urdf/cr5/cr5_controller.xacro (robot description, xacro)
@@ -12,9 +12,10 @@
         </joint>
     </xacro:macro>
-    <xacro:macro name="cr5_ros2_control" params="prefix:='' ">
+    <xacro:macro name="cr5_ros2_control" params="prefix:='' mujoco_model">
         <ros2_control name="${prefix}cr5_system" type="system">
             <hardware>
                 <plugin>mujoco_ros2_control/MujocoSystemInterface</plugin>
-                <param name="mujoco_model">$(find dobot_mujoco_integration)/scenes/main_scene.xml</param>
+                <param name="mujoco_model">${mujoco_model}</param>
+                <param name="auto_register_cameras">false</param>
             </hardware>
             <xacro:cr5_joint_interface joint_name="${prefix}joint_1" />

File: workspace/src/dobot_description/urdf/cr5/cr5_macro.xacro (robot description, xacro)
@@ -1,5 +1,5 @@
 <?xml version="1.0"?>
 <robot xmlns:xacro="http://www.ros.org/wiki/xacro">
-    <xacro:macro name="cr5_robot" params="prefix:=^|'' package_name:='cr5_description'">
+    <xacro:macro name="cr5_robot" params="prefix:=^|''">
         <!-- Base Link -->
         <link name="${prefix}base_link">
@@ -13,11 +13,11 @@
                 <origin xyz="0 0 0" rpy="0 0 0" />
                 <geometry>
-                    <mesh filename="package://${package_name}/meshes/visual/base.STL" />
-                </geometry>
-            </visual>
-            <collision>
-                <origin xyz="0 0 0" rpy="0 0 0" />
-                <geometry>
-                    <mesh filename="package://${package_name}/meshes/collision/base.STL" />
+                    <mesh filename="package://dobot_description/meshes/cr5/visual/base.STL" />
+                </geometry>
+            </visual>
+            <collision>
+                <origin xyz="0 0 0" rpy="0 0 0" />
+                <geometry>
+                    <mesh filename="package://dobot_description/meshes/cr5/collision/base.STL" />
                 </geometry>
             </collision>
@@ -42,11 +42,11 @@
                 <origin xyz="0 0 0" rpy="0 0 0" />
                 <geometry>
-                    <mesh filename="package://${package_name}/meshes/visual/link_1.STL" />
-                </geometry>
-            </visual>
-            <collision>
-                <origin xyz="0 0 0" rpy="0 0 0" />
-                <geometry>
-                    <mesh filename="package://${package_name}/meshes/collision/link_1.STL" />
+                    <mesh filename="package://dobot_description/meshes/cr5/visual/link_1.STL" />
+                </geometry>
+            </visual>
+            <collision>
+                <origin xyz="0 0 0" rpy="0 0 0" />
+                <geometry>
+                    <mesh filename="package://dobot_description/meshes/cr5/collision/link_1.STL" />
                 </geometry>
             </collision>
@@ -71,11 +71,11 @@
                 <origin xyz="0 0 0" rpy="0 0 0" />
                 <geometry>
-                    <mesh filename="package://${package_name}/meshes/visual/link_2.STL" />
-                </geometry>
-            </visual>
-            <collision>
-                <origin xyz="0 0 0" rpy="0 0 0" />
-                <geometry>
-                    <mesh filename="package://${package_name}/meshes/collision/link_2.STL" />
+                    <mesh filename="package://dobot_description/meshes/cr5/visual/link_2.STL" />
+                </geometry>
+            </visual>
+            <collision>
+                <origin xyz="0 0 0" rpy="0 0 0" />
+                <geometry>
+                    <mesh filename="package://dobot_description/meshes/cr5/collision/link_2.STL" />
                 </geometry>
             </collision>
@@ -100,11 +100,11 @@
                 <origin xyz="0 0 0" rpy="0 0 0" />
                 <geometry>
-                    <mesh filename="package://${package_name}/meshes/visual/link_3.STL" />
-                </geometry>
-            </visual>
-            <collision>
-                <origin xyz="0 0 0" rpy="0 0 0" />
-                <geometry>
-                    <mesh filename="package://${package_name}/meshes/collision/link_3.STL" />
+                    <mesh filename="package://dobot_description/meshes/cr5/visual/link_3.STL" />
+                </geometry>
+            </visual>
+            <collision>
+                <origin xyz="0 0 0" rpy="0 0 0" />
+                <geometry>
+                    <mesh filename="package://dobot_description/meshes/cr5/collision/link_3.STL" />
                 </geometry>
             </collision>
@@ -129,11 +129,11 @@
                 <origin xyz="0 0 0" rpy="0 0 0" />
                 <geometry>
-                    <mesh filename="package://${package_name}/meshes/visual/link_4.STL" />
-                </geometry>
-            </visual>
-            <collision>
-                <origin xyz="0 0 0" rpy="0 0 0" />
-                <geometry>
-                    <mesh filename="package://${package_name}/meshes/collision/link_4.STL" />
+                    <mesh filename="package://dobot_description/meshes/cr5/visual/link_4.STL" />
+                </geometry>
+            </visual>
+            <collision>
+                <origin xyz="0 0 0" rpy="0 0 0" />
+                <geometry>
+                    <mesh filename="package://dobot_description/meshes/cr5/collision/link_4.STL" />
                 </geometry>
             </collision>
@@ -158,11 +158,11 @@
                 <origin xyz="0 0 0" rpy="0 0 0" />
                 <geometry>
-                    <mesh filename="package://${package_name}/meshes/visual/link_5.STL" />
-                </geometry>
-            </visual>
-            <collision>
-                <origin xyz="0 0 0" rpy="0 0 0" />
-                <geometry>
-                    <mesh filename="package://${package_name}/meshes/collision/link_5.STL" />
+                    <mesh filename="package://dobot_description/meshes/cr5/visual/link_5.STL" />
+                </geometry>
+            </visual>
+            <collision>
+                <origin xyz="0 0 0" rpy="0 0 0" />
+                <geometry>
+                    <mesh filename="package://dobot_description/meshes/cr5/collision/link_5.STL" />
                 </geometry>
             </collision>
@@ -187,11 +187,11 @@
                 <origin xyz="0 0 0" rpy="0 0 0" />
                 <geometry>
-                    <mesh filename="package://${package_name}/meshes/visual/link_6.STL" />
-                </geometry>
-            </visual>
-            <collision>
-                <origin xyz="0 0 0" rpy="0 0 0" />
-                <geometry>
-                    <mesh filename="package://${package_name}/meshes/collision/link_6.STL" />
+                    <mesh filename="package://dobot_description/meshes/cr5/visual/link_6.STL" />
+                </geometry>
+            </visual>
+            <collision>
+                <origin xyz="0 0 0" rpy="0 0 0" />
+                <geometry>
+                    <mesh filename="package://dobot_description/meshes/cr5/collision/link_6.STL" />
                 </geometry>
             </collision>
