Commit message: added moveit configuration

File: workspace/src/dobot_description/urdf/cr5/cr5_macro.xacro (robot description, xacro)
@@ -199,8 +199,8 @@
         <joint name="${prefix}tcp_joint" type="fixed">
             <parent link="${prefix}link_6" />
-            <child link="${prefix}tcp_link" />
+            <child link="${prefix}flange" />
             <origin xyz="0 0 0.01" rpy="0 0 0" />
         </joint>
-        <link name="${prefix}tcp_link" />
+        <link name="${prefix}flange" />
     </xacro:macro>
 </robot>

Commit message: bug fixes

File: workspace/src/dobot_description/urdf/cr5/cr5_macro.xacro (robot description, xacro)
@@ -199,5 +199,5 @@
             <parent link="${prefix}link_6" />
             <child link="${prefix}flange" />
-            <origin xyz="0 0 0.01" rpy="0 0 0" />
+            <origin xyz="0 0 0.0" rpy="0 0 0" />
         </joint>
         <link name="${prefix}flange" />
