Commit message: C3: split packages by responsibility

File: workspace/src/robots/dobot_cr5_description/urdf/cr5/cr5.urdf.xacro (robot description, xacro)
@@ -2,5 +2,5 @@
 <robot xmlns:xacro="http://www.ros.org/wiki/xacro" name="cr5">
     <xacro:arg name="prefix" default="" />
-    <xacro:include filename="$(find dobot_description)/urdf/cr5/cr5_macro.xacro" />
+    <xacro:include filename="$(find dobot_cr5_description)/urdf/cr5/cr5_macro.xacro" />
     <link name="world" />
     <joint name="$(arg prefix)world_to_base_joint" type="fixed">

File: workspace/src/robots/dobot_cr5_description/urdf/cr5/cr5_macro.xacro (robot description, xacro)
@@ -13,11 +13,11 @@
                 <origin xyz="0 0 0" rpy="0 0 0" />
                 <geometry>
-                    <mesh filename="package://dobot_description/meshes/cr5/visual/base.STL" />
-                </geometry>
-            </visual>
-            <collision>
-                <origin xyz="0 0 0" rpy="0 0 0" />
-                <geometry>
-                    <mesh filename="package://dobot_description/meshes/cr5/collision/base.STL" />
+                    <mesh filename="package://dobot_cr5_description/meshes/cr5/visual/base.STL" />
+                </geometry>
+            </visual>
+            <collision>
+                <origin xyz="0 0 0" rpy="0 0 0" />
+                <geometry>
+                    <mesh filename="package://dobot_cr5_description/meshes/cr5/collision/base.STL" />
                 </geometry>
             </collision>
@@ -42,11 +42,11 @@
                 <origin xyz="0 0 0" rpy="0 0 0" />
                 <geometry>
-                    <mesh filename="package://dobot_description/meshes/cr5/visual/link_1.STL" />
-                </geometry>
-            </visual>
-            <collision>
-                <origin xyz="0 0 0" rpy="0 0 0" />
-                <geometry>
-                    <mesh filename="package://dobot_description/meshes/cr5/collision/link_1.STL" />
+                    <mesh filename="package://dobot_cr5_description/meshes/cr5/visual/link_1.STL" />
+                </geometry>
+            </visual>
+            <collision>
+                <origin xyz="0 0 0" rpy="0 0 0" />
+                <geometry>
+                    <mesh filename="package://dobot_cr5_description/meshes/cr5/collision/link_1.STL" />
                 </geometry>
             </collision>
@@ -71,11 +71,11 @@
                 <origin xyz="0 0 0" rpy="0 0 0" />
                 <geometry>
-                    <mesh filename="package://dobot_description/meshes/cr5/visual/link_2.STL" />
-                </geometry>
-            </visual>
-            <collision>
-                <origin xyz="0 0 0" rpy="0 0 0" />
-                <geometry>
-                    <mesh filename="package://dobot_description/meshes/cr5/collision/link_2.STL" />
+                    <mesh filename="package://dobot_cr5_description/meshes/cr5/visual/link_2.STL" />
+                </geometry>
+            </visual>
+            <collision>
+                <origin xyz="0 0 0" rpy="0 0 0" />
+                <geometry>
+                    <mesh filename="package://dobot_cr5_description/meshes/cr5/collision/link_2.STL" />
                 </geometry>
             </collision>
@@ -100,11 +100,11 @@
                 <origin xyz="0 0 0" rpy="0 0 0" />
                 <geometry>
-                    <mesh filename="package://dobot_description/meshes/cr5/visual/link_3.STL" />
-                </geometry>
-            </visual>
-            <collision>
-                <origin xyz="0 0 0" rpy="0 0 0" />
-                <geometry>
-                    <mesh filename="package://dobot_description/meshes/cr5/collision/link_3.STL" />
+                    <mesh filename="package://dobot_cr5_description/meshes/cr5/visual/link_3.STL" />
+                </geometry>
+            </visual>
+            <collision>
+                <origin xyz="0 0 0" rpy="0 0 0" />
+                <geometry>
+                    <mesh filename="package://dobot_cr5_description/meshes/cr5/collision/link_3.STL" />
                 </geometry>
             </collision>
@@ -129,11 +129,11 @@
                 <origin xyz="0 0 0" rpy="0 0 0" />
                 <geometry>
-                    <mesh filename="package://dobot_description/meshes/cr5/visual/link_4.STL" />
-                </geometry>
-            </visual>
-            <collision>
-                <origin xyz="0 0 0" rpy="0 0 0" />
-                <geometry>
-                    <mesh filename="package://dobot_description/meshes/cr5/collision/link_4.STL" />
+                    <mesh filename="package://dobot_cr5_description/meshes/cr5/visual/link_4.STL" />
+                </geometry>
+            </visual>
+            <collision>
+                <origin xyz="0 0 0" rpy="0 0 0" />
+                <geometry>
+                    <mesh filename="package://dobot_cr5_description/meshes/cr5/collision/link_4.STL" />
                 </geometry>
             </collision>
@@ -158,11 +158,11 @@
                 <origin xyz="0 0 0" rpy="0 0 0" />
                 <geometry>
-                    <mesh filename="package://dobot_description/meshes/cr5/visual/link_5.STL" />
-                </geometry>
-            </visual>
-            <collision>
-                <origin xyz="0 0 0" rpy="0 0 0" />
-                <geometry>
-                    <mesh filename="package://dobot_description/meshes/cr5/collision/link_5.STL" />
+                    <mesh filename="package://dobot_cr5_description/meshes/cr5/visual/link_5.STL" />
+                </geometry>
+            </visual>
+            <collision>
+                <origin xyz="0 0 0" rpy="0 0 0" />
+                <geometry>
+                    <mesh filename="package://dobot_cr5_description/meshes/cr5/collision/link_5.STL" />
                 </geometry>
             </collision>
@@ -187,11 +187,11 @@
                 <origin xyz="0 0 0" rpy="0 0 0" />
                 <geometry>
-                    <mesh filename="package://dobot_description/meshes/cr5/visual/link_6.STL" />
-                </geometry>
-            </visual>
-            <collision>
-                <origin xyz="0 0 0" rpy="0 0 0" />
-                <geometry>
-                    <mesh filename="package://dobot_description/meshes/cr5/collision/link_6.STL" />
+                    <mesh filename="package://dobot_cr5_description/meshes/cr5/visual/link_6.STL" />
+                </geometry>
+            </visual>
+            <collision>
+                <origin xyz="0 0 0" rpy="0 0 0" />
+                <geometry>
+                    <mesh filename="package://dobot_cr5_description/meshes/cr5/collision/link_6.STL" />
                 </geometry>
             </collision>
